File: IRBlaster.brd (EAGLE design)
At the start: 70.8 x 58.4 mm, 12 parts, among them T4 2N3904, T5 2N3904, T6 2N3904

Commit message: Add PCB Files
Parts:
- R1, R3, R5: value (none) -> 1K
- R2, R4, R6: value (none) -> 100
- moved IR1 12.7 mm to (69.8, 3.81), turned to 270 degrees
- moved U$1 7.62 mm to (31.8, 24.1)
Connections:
- removed net N$13: R6.2, T6.1
- removed net N$7: R5.1, SV1.2
- net N$10: now also R3.1; no longer SV1.3
- net N$11: now also SV1.3; no longer R4.2
- net N$12: now also R5.1, R6.2, SV1.2; no longer SV1.1
- net N$14: now also SV1.1, T6.1; no longer R2.1
- net N$5: now also R4.2, SV1.4; no longer R1.1, SV1.6
- net N$6: now also R2.2, SV1.6; no longer R3.1, SV1.4
- net N$8: now also R1.1; no longer SV1.5
- net N$9: now also SV1.5; no longer R2.2
- net VCC: now also R2.1, R4.1
Routing:
- net VCC: track 36.6 -> 174.5 mm
- net GND: track 113.9 -> 0.00 mm
- net N$7: track 55.2 -> 0.00 mm, vias 4 -> 0
- net N$10: track 47.8 -> 7.93 mm
- net N$1: track 78.5 -> 43.4 mm
- net N$8: track 39.2 -> 10.8 mm
- net N$12: track 46.4 -> 73.3 mm
- net N$3: track 17.1 -> 37.0 mm
- net N$14: track 0.00 -> 14.3 mm
- net N$13: track 13.8 -> 0.00 mm
- net VCC/2: track 17.0 -> 28.3 mm
- net N$6: track 33.2 -> 25.4 mm
- net N$4: track 19.7 -> 25.3 mm
- net N$5: track 29.5 -> 26.0 mm
- net N$9: track 11.7 -> 13.7 mm
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- added copper zone on layer 16, net GND
- removed copper zone on layer 16, net N$15
Other:
- board text added: "IR Leds Emitters"
- board text added: "IRBlaster - v0.2"
- board text removed: "External IR Emitters (3)"
- board text removed: "IRBlaster - v0.1"
